Commit message: no db

File: catkin_ws/src/my_robot/urdf/my_robot.xacro (robot description, xacro)
@@ -176,4 +176,11 @@
     </visual>
   </link>
+  <link name="camera_link_optical">
+  </link>
+  <joint name="camera_optical_joint" type="fixed">
+    <origin xyz="0 0 0" rpy="-1.5707 0 -1.5707"/>
+    <parent link="camera"/>
+    <child link="camera_link_optical"/>
+  </joint>
   <joint type="fixed" name="hokuyo_joint">
     <origin xyz="0.15 0.0 0.1" rpy="0 0 0"/>
